Commit message: Migrate simulator to Webots

File: description/gps.xacro (robot description, xacro)
@@ -8,12 +8,3 @@
     <link name="gps">
     </link>
-    <gazebo reference="gps">
-        <sensor name="gps" type="navsat">
-            <gz_frame_id>gps</gz_frame_id>
-            <always_on>1</always_on>
-            <update_rate>5</update_rate>
-            <topic>gps/fix</topic>
-        </sensor>
-        <material>Gazebo/Black</material>
-    </gazebo>
 </robot>

File: description/imu.xacro (robot description, xacro)
@@ -8,14 +8,3 @@
     <link name="imu">
     </link>
-    <gazebo reference="imu">
-        <sensor name="imu" type="imu">
-            <gz_frame_id>imu</gz_frame_id>
-            <!-- not possible to disable orientation via SDF, we will skip it during fusion-->
-            <always_on>1</always_on>
-            <update_rate>50</update_rate>
-            <visualize>true</visualize>
-            <topic>imu/data_raw</topic>
-        </sensor>
-        <material>Gazebo/Red</material>
-    </gazebo>
 </robot>

File: description/robot.urdf.xacro (robot description, xacro)
@@ -12,6 +12,6 @@
         <xacro:include filename="ros2_control.xacro" />
     </xacro:if>
-    <xacro:unless value="$(arg use_ros2_control)">
-        <xacro:include filename="gazebo_control.xacro" />
-    </xacro:unless>
+    <xacro:if value="$(arg sim_mode)">
+        <xacro:include filename="webots_control.xacro" />
+    </xacro:if>
 </robot>

File: description/robot_core.xacro (robot description, xacro)
@@ -41,10 +41,4 @@
     <link name="base_link">
     </link>
-    <gazebo>
-        <plugin filename="gz-sim-pose-publisher-system" name="gz::sim::systems::PosePublisher">
-            <use_pose_vector_msg>true</use_pose_vector_msg>
-            <publish_nested_model_pose>true</publish_nested_model_pose>
-        </plugin>
-    </gazebo>
     <!-- BASE_FOOTPRINT LINK -->
     <joint name="base_footprint_joint" type="fixed">
@@ -79,7 +73,4 @@
         </xacro:inertial_box>
     </link>
-    <gazebo reference="chassis">
-        <material>Gazebo/Orange</material>
-    </gazebo>
     <!-- CHARGING PORT LINK -->
     <xacro:property name="charging_port_radius" value="0.01"/>
@@ -106,7 +97,4 @@
         </xacro:inertial_sphere>
     </link>
-    <gazebo reference="charging_port">
-        <material>Gazebo/Green</material>
-    </gazebo>
     <!-- LEFT WHEEL LINK -->
     <joint name="left_wheel_joint" type="continuous">
@@ -133,16 +121,4 @@
         </xacro:inertial_cylinder>
     </link>
-    <gazebo reference="left_wheel">
-        <material>Gazebo/Blue</material>
-        <mu1 value="1.0"/>
-        <mu2 value="1.0"/>
-        <kp value="10000000.0" />
-        <kd value="1.0" />
-        <fdir1 value="1 0 0"/>
-        <minDepth>0.005</minDepth>
-        <maxVel>1.0</maxVel>
-        <slip1>0.0</slip1>
-        <slip2>0.0</slip2>
-    </gazebo>
     <!-- RIGHT WHEEL LINK -->
     <joint name="right_wheel_joint" type="continuous">
@@ -169,16 +145,4 @@
         </xacro:inertial_cylinder>
     </link>
-    <gazebo reference="right_wheel">
-        <material>Gazebo/Blue</material>
-        <mu1 value="1.0"/>
-        <mu2 value="1.0"/>
-        <kp value="10000000.0" />
-        <kd value="1.0" />
-        <fdir1 value="1 0 0"/>
-        <minDepth>0.005</minDepth>
-        <maxVel>1.0</maxVel>
-        <slip1>0.0</slip1>
-        <slip2>0.0</slip2>
-    </gazebo>
     <!-- MOWER LINK -->
     <joint name="mower_joint" type="continuous">
@@ -204,9 +168,4 @@
         </xacro:inertial_cylinder>
     </link>
-    <gazebo reference="mower">
-        <material>Gazebo/Red</material>
-        <mu1 value="0.5"/>
-        <mu2 value="0.5"/>
-    </gazebo>
     <!-- LEFT CASTER WHEEL LINK -->
     <!-- Caster Swivel -->
@@ -222,7 +181,4 @@
         </xacro:inertial_sphere>
     </link>
-    <gazebo reference="left_caster_swivel">
-        <material>Gazebo/Black</material>
-    </gazebo>
     <joint name="left_caster_wheel_joint" type="continuous">
         <parent link="left_caster_swivel"/>
@@ -247,11 +203,4 @@
         </xacro:inertial_sphere>
     </link>
-    <gazebo reference="left_caster_wheel">
-        <material>Gazebo/Black</material>
-        <mu1 value="0.001"/>
-        <mu2 value="0.001"/>
-        <kp value="10000.0" />
-        <kd value="1.0" />
-    </gazebo>
     <!-- RIGHT CASTER WHEEL LINK -->
     <!-- Caster Swivel -->
@@ -267,7 +216,4 @@
         </xacro:inertial_sphere>
     </link>
-    <gazebo reference="right_caster_swivel">
-        <material>Gazebo/Black</material>
-    </gazebo>
     <joint name="right_caster_wheel_joint" type="continuous">
         <parent link="right_caster_swivel"/>
@@ -292,17 +238,3 @@
         </xacro:inertial_sphere>
     </link>
-    <gazebo reference="right_caster_wheel">
-        <material>Gazebo/Black</material>
-        <mu1 value="0.001"/>
-        <mu2 value="0.001"/>
-        <kp value="10000.0" />
-        <kd value="1.0" />
-    </gazebo>
-    <!-- Global collision settings -->
-    <gazebo>
-        <self_collide>0</self_collide>
-        <collision_detector>bullet</collision_detector>
-        <static>0</static>
-        <gravity>1</gravity>
-    </gazebo>
 </robot>

Commit message: Stabilize FusionCore Webots simulation

File: description/gps.xacro (robot description, xacro)
@@ -3,8 +3,8 @@
     <joint name="gps_joint" type="fixed">
         <parent link="base_link"/>
-        <child link="gps"/>
+        <child link="gnss_link"/>
         <origin xyz="${robot['gps']['antenna']['offset'][0]} ${robot['gps']['antenna']['offset'][1]} ${robot['gps']['antenna']['offset'][2]}" rpy="0 0 0"/>
     </joint>
-    <link name="gps">
+    <link name="gnss_link">
     </link>
 </robot>
